File: Heart Rate Headphones.sch (EAGLE design)
At the start: 1 part, among them P1 SEN-11574

Commit message: ADC converter
Parts:
- removed P1: SEN-11574, SEN-11574:SEN-11574
- added X1: RASPI_BOARD_AB_F, raspberrypi_bastelstube_v13:RASPI_BOARD_AB_F
Other:
- note added: "Heart Rate Headphones"
Changed lines of the file:
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@@
 <parts>
 <part name="FRAME1" library="dframes" deviceset="DINA3_L" device=""/>
-<part name="P1" library="SEN-11574" deviceset="SEN-11574" device=""/>
+<part name="X1" library="raspberrypi_bastelstube_v13" deviceset="RASPI_BOARD_AB" device="_F"/>
 </parts>
 <sheets>
 <sheet>
 <plain>
+<text x="127" y="-114.3" size="1.778" layer="91">Heart Rate Headphones</text>
 </plain>
 <instances>
-<instance part="FRAME1" gate="G$1" x="-264.16" y="-20.32"/>
-<instance part="FRAME1" gate="G$2" x="2.54" y="-20.32"/>
-<instance part="FRAME1" gate="G$3" x="-63.5" y="-20.32"/>
-<instance part="P1" gate="G$1" x="-121.92" y="93.98"/>
+<instance part="FRAME1" gate="G$1" x="-187.96" y="-134.62"/>
+<instance part="FRAME1" gate="G$2" x="78.74" y="-134.62"/>
+<instance part="FRAME1" gate="G$3" x="12.7" y="-134.62"/>
+<instance part="X1" gate="G$1" x="0" y="55.88"/>
 </instances>
 <busses>
