File: FYDE PCB Rough.brd (EAGLE design)
At the start: 29.2 x 22.9 mm, 39 parts, among them CN1 USBA_FEMALE, P1 SEN-11574, T1 MMUN2133LT1G, U1 TPS61030RSAR, X2 3.5mm, X4 RASPI_BOARD_B+_FP

Commit message: Add files via upload
updated, more concise
Parts:
- removed X4: RASPI_BOARD_B+_FP, raspberrypi_bastelstube_v13:RASPI_BOARD_B+_FULL_PAD
- added X3: 3.5mm, microbuilder:TERMBLOCK_1X2-3.5MM
- X1: value (none) -> RASPI_BOARD_B+_FP; device microbuilder:TERMBLOCK_1X2-3.5MM -> raspberrypi_bastelstube_v13:RASPI_BOARD_B+_FULL_PAD
- X2: value 3.5mm -> (none)
- moved B1 141.8 mm to (-20.6, -128.3)
- moved LED2 141.8 mm to (2.73, -138.1)
- moved R1 141.8 mm to (-12.4, -127.3)
- moved R13 141.8 mm to (-14.1, -131.8)
- moved R20 141.8 mm to (-17.4, -134.1)
- moved U$25 141.8 mm to (0.13, -133.5)
- moved U$33 141.8 mm to (-12.8, -139.2)
- moved C1 141.8 mm to (-12.4, -124.6)
- moved C2 141.8 mm to (-4.06, -133.0)
- moved C3 141.8 mm to (-3.30, -137.2)
- moved C4 141.8 mm to (-14.6, -124.6)
- moved C6 141.8 mm to (-6.48, -137.2)
- moved CN1 141.8 mm to (6.73, -128.0)
- moved FID1 141.8 mm to (3.94, -124.0)
- moved FID2 141.8 mm to (-20.9, -122.7)
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Connections:
- net 3V3: now also X1.1; no longer X4.1
- net 5.0V: now also X2.2; no longer X1.2
- net 5V0: now also X1.2; no longer X4.2
- net GND: now also X1.6, X3.1; no longer X1.1, X4.6
- net VBAT: now also X3.2; no longer X2.2
Routing:
- net N$7: track 0.00 -> 27.9 mm
Other:
- board size 29.2 x 22.9 mm -> 123.2 x 205.4 mm

Commit message: updated; includes Power Booster custom library
Parts:
- removed B1: 1.8-5V, microbuilder:JSTPH2
- removed C1: 10uF, microbuilder:0805-NO
- removed C2: 2.2uF, microbuilder:0805-NO
- removed C3, C6: 100uF, rcl:C1210
- removed C4: 0.1uF, microbuilder:0805-NO
- removed CN1: USBA_FEMALE, microbuilder:USB_HOST-PTH
- removed FID1, FID2, FID3: FIDUCIAL"", microbuilder:FIDUCIAL_1MM
- removed JP1: (no value), adafruit:1X06-CLEANBIG
- removed L1: 6.8uH, microbuilder:INDUCTOR_8X8MM
- removed LED1: RED, microbuilder:CHIPLED_0805_NOOUTLINE
- removed LED2: GREEN, microbuilder:CHIPLED_0805_NOOUTLINE
- removed R1, R3: 1.87M, microbuilder:_0805MP
- removed R10, R12: 49.9K 1%, microbuilder:0805-NO
- removed R11: 75K 1%, microbuilder:0805-NO
- removed R13, R4: 200K, microbuilder:0805-NO
- removed R2: 340K, microbuilder:_0805MP
- removed R20, R5: 1K, microbuilder:0805-NO
- removed R9: 43K 1%, microbuilder:0805-NO
- removed T1: MMUN2133LT1G, transistor:SC59-BEC
- removed U$10, U$11: MOUNTINGHOLE2.5, microbuilder:MOUNTINGHOLE_2.5_PLATED
- removed U$12, U$26: (no value), microbuilder:SYMBOL_MINUS
- removed U$13, U$25: (no value), microbuilder:SYMBOL_PLUS
- removed U$28, U$33: (no value), microbuilder:ADAFRUIT_5MM
- removed U1: TPS61030RSAR, microbuilder:PVQFN-16
- removed X2: (no value), microbuilder:TERMBLOCK_1X2-3.5MM
- removed X3: 3.5mm, microbuilder:TERMBLOCK_1X2-3.5MM
- added U$1: ADAFRUITPOWERBOOSTER(FYDE), Adafruit-PowerBoost-FYDE:ADAFRUITPOWERBOOSTER(FYDE)
Connections:
- removed net 5.0V: C2.1, C3.1, C6.1, CN1.VBUS, JP1.6, R11.2, R3.2, R5.1, R9.2, U1.1, U1.15, U1.16, X2.2
- removed net D+: CN1.D+, R11.1, R12.1
- removed net D-: CN1.D-, R10.1, R9.1
- removed net ENABLE: JP1.3, R13.2, U1.11
- removed net LBO: JP1.4, T1.B, U1.12
- removed net VBAT: B1.2, C1.1, C4.1, JP1.1, L1.P$1, R1.2, R13.1, T1.E, U1.8, X3.2
- net GND: no longer B1.1, C1.2, C2.2, C3.2, C4.2, C6.2, CN1.GND, JP1.2, JP1.5, LED1.C, LED2.C, R10.2, R12.2, R2.1, R4.1, U1.10, U1.13, U1.5, U1.6, U1.7, U1.P$18, U1.P$19, U1.P$20, U1.P$21, U1.P$22, U1.THERMAL, X2.1, X3.1
- net N$1: now also U$1.6; no longer L1.P$2, U1.3, U1.4
- net N$2: now also U$1.5; no longer LED1.A, R20.1
- net N$3: now also U$1.4; no longer R1.1, R2.2, U1.9
- net N$4: now also U$1.3; no longer LED2.A, R5.2
- net N$5: now also U$1.2; no longer R3.1, R4.2, U1.14
- net N$6: now also U$1.1; no longer R20.2, T1.C
Routing:
- net VBAT: track 38.6 -> 0.00 mm, vias 1 -> 0
- net 5.0V: track 29.4 -> 0.00 mm
- net LBO: track 27.8 -> 0.00 mm, vias 3 -> 0
- net ENABLE: track 18.6 -> 0.00 mm, vias 2 -> 0
- net D+: track 12.6 -> 0.00 mm
- net N$5: track 9.32 -> 0.00 mm
- net GND: track 8.02 -> 0.00 mm, vias 20 -> 0
- net D-: track 5.78 -> 0.00 mm
- net N$3: track 4.02 -> 0.00 mm
- net N$6: track 2.83 -> 0.00 mm
- net N$4: track 2.01 -> 0.00 mm
- net N$2: track 2.01 -> 0.00 mm
- removed copper zone on layer 1, net 5.0V
- removed copper zone on layer 1, net GND
- removed copper zone on layer 16, net GND
- removed copper zone on layer 1, net N$1
- removed copper zone on layer 1, net VBAT
Other:
- board size 123.2 x 205.4 mm -> 99 x 65.7 mm
- board text removed: "1000"
- board text removed: "1000mA+ from 1.8-5V"
- board text removed: "3.2V Low Batt"
- board text removed: "5.2V output"
- board text removed: "5V"
- board text removed: "Bat"
- board text removed: "EN"
- board text removed: "GND"
- board text removed: "LB"
- board text removed: "LOW"
- board text removed: "PWR"
- board text removed: "Power Boost"
- board text removed: "PowerBoost 1000 Basic"
- board text removed: "TPS61030 DC Boost"
- board text removed: "adafruit"
- board text removed: "iOS 1A Charge Resistors"

Commit message: Add files via upload
Parts:
- added U1: MCU-MCP3008-I/P(DIP16-7.62MM), MCU-MCP3008-I_P_DIP16-7.62MM_:DIP16-2.54-19.2X7.62MM
- moved U$1 52.1 mm to (12.7, 17.8)
- moved P1 39.2 mm to (68.6, 36.8)
Connections:
- removed net N$1: U$1.6
- removed net N$2: U$1.5
- removed net N$3: U$1.4
- removed net N$4: U$1.3
- removed net N$5: U$1.2
- removed net N$6: U$1.1
Changed lines of the file:
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@@
 </autorouter>
 <elements>
-<element name="P1" library="SEN-11574" package="XDCR_SEN-11574" value="SEN-11574" x="102.87" y="55.88">
-<attribute name="AVAILABILITY" value="Unavailable" x="102.87" y="55.88" size="1.778" layer="27" display="off"/>
-<attribute name="DESCRIPTION" value=" PULSE SENSOR FOR ARDUINO " x="102.87" y="55.88" size="1.778" layer="27" display="off"/>
-<attribute name="MF" value="SparkFun" x="102.87" y="55.88" size="1.778" layer="27" display="off"/>
-<attribute name="MP" value="SEN-11574" x="102.87" y="55.88" size="1.778" layer="27" display="off"/>
-<attribute name="PACKAGE" value="None" x="102.87" y="55.88" size="1.778" layer="27" display="off"/>
-<attribute name="PRICE" value="None" x="102.87" y="55.88" size="1.778" layer="27" display="off"/>
+<element name="P1" library="SEN-11574" package="XDCR_SEN-11574" value="SEN-11574" x="68.58" y="36.83">
+<attribute name="AVAILABILITY" value="Unavailable" x="68.58" y="36.83" size="1.778" layer="27" display="off"/>
+<attribute name="DESCRIPTION" value=" PULSE SENSOR FOR ARDUINO " x="68.58" y="36.83" size="1.778" layer="27" display="off"/>
+<attribute name="MF" value="SparkFun" x="68.58" y="36.83" size="1.778" layer="27" display="off"/>
+<attribute name="MP" value="SEN-11574" x="68.58" y="36.83" size="1.778" layer="27" display="off"/>
+<attribute name="PACKAGE" value="None" x="68.58" y="36.83" size="1.778" layer="27" display="off"/>
+<attribute name="PRICE" value="None" x="68.58" y="36.83" size="1.778" layer="27" display="off"/>
 </element>
 <element name="X1" library="raspberrypi_bastelstube_v13" package="RASPI_BOARD_B+_FULL_PAD" value="RASPI_BOARD_B+_FP" x="6.35" y="5.08"/>
-<element name="U$1" library="Adafruit-PowerBoost-FYDE" package="ADAFRUITPOWERBOOSTER(FYDE)" value="ADAFRUITPOWERBOOSTER(FYDE)" x="12.7" y="-34.29"/>
+<element name="U$1" library="Adafruit-PowerBoost-FYDE" package="ADAFRUITPOWERBOOSTER(FYDE)" value="ADAFRUITPOWERBOOSTER(FYDE)" x="12.7" y="17.78"/>
+<element name="U1" library="MCU-MCP3008-I_P_DIP16-7.62MM_" package="DIP16-2.54-19.2X7.62MM" value="MCU-MCP3008-I/P(DIP16-7.62MM)" x="35.56" y="-34.29">
+<attribute name="AVAILABILITY" value="Unavailable" x="35.56" y="-34.29" size="1.778" layer="27" display="off"/>
+<attribute name="DESCRIPTION" value=" 10 Bit Analog to Digital Converter 4, 8 Input 1 SAR 16-PDIP " x="35.56" y="-34.29" size="1.778" layer="27" display="off"/>
+<attribute name="MF" value="Microchip" x="35.56" y="-34.29" size="1.778" layer="27" display="off"/>
+<attribute name="MP" value="MCP3008-I/P" x="35.56" y="-34.29" size="1.778" layer="27" display="off"/>
+<attribute name="PACKAGE" value="DIP-16 Microchip" x="35.56" y="-34.29" size="1.778" layer="27" display="off"/>
+<attribute name="PRICE" value="None" x="35.56" y="-34.29" size="1.778" layer="27" display="off"/>
+</element>
 </elements>
 <signals>
@@
 <contactref element="P1" pad="3"/>
 <contactref element="X1" pad="6"/>
-<wire x1="19.8" y1="58.85" x2="102.87" y2="58.42" width="0" layer="19" extent="1-1"/>
+<wire x1="19.8" y1="58.85" x2="68.58" y2="39.37" width="0" layer="19" extent="1-1"/>
 </signal>
 <signal name="5V0">
@@
 <wire x1="64.77" y1="53.34" x2="64.77" y2="45.72" width="0.1524" layer="1"/>
 </signal>
-<signal name="N$1">
-<contactref element="U$1" pad="6"/>
-</signal>
-<signal name="N$2">
-<contactref element="U$1" pad="5"/>
-</signal>
-<signal name="N$3">
-<contactref element="U$1" pad="4"/>
-</signal>
-<signal name="N$4">
-<contactref element="U$1" pad="3"/>
-</signal>
-<signal name="N$5">
-<contactref element="U$1" pad="2"/>
-</signal>
-<signal name="N$6">
-<contactref element="U$1" pad="1"/>
-</signal>
 </signals>
