File: FYDE PCB Rough.brd (EAGLE design)
At the start: 65 x 56.1 mm, 4 parts, among them P1 SEN-11574, U1 MCU-MCP3008-I/P(DIP16-7.62MM), X1 RASPI_BOARD_B+_HDC

Commit message: Add files via upload
new powerbooster (with library)
Parts:
- removed U$1: ADAFRUITPOWERBOOSTER(FYDE), Adafruit-PowerBoost-FYDE:ADAFRUITPOWERBOOSTER(FYDE)
- added J1: (no value), SparkFun-Connectors:JST-2-SMD
- added U$2: MT3608, MT3608:MT3608
Connections:
- net +3V3A: now also J1.2, U$2.P$1
- net +5V: now also U$2.P$3
- net GND: now also J1.1, U$2.P$2, U$2.P$4
Routing:
- net +5V: track 11.9 -> 65.6 mm, vias 0 -> 2
- net +3V3A: track 13.6 -> 55.1 mm, vias 0 -> 2
- net GND: track 0.00 -> 18.7 mm
Other:
- outline, holes or cut-outs redrawn
Changed lines of the file:
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@@
 <layer number="112" name="tSilk" color="7" fill="1" visible="no" active="yes"/>
 <layer number="113" name="ReferenceLS" color="7" fill="1" visible="no" active="no"/>
+<layer number="114" name="Badge_Outline" color="7" fill="1" visible="yes" active="yes"/>
+<layer number="115" name="ReferenceISLANDS" color="7" fill="1" visible="yes" active="yes"/>
 <layer number="116" name="Patch_BOT" color="9" fill="4" visible="no" active="yes"/>
 <layer number="118" name="Rect_Pads" color="7" fill="1" visible="no" active="no"/>
@@
 <wire x1="4.318" y1="41.656" x2="2.54" y2="43.434" width="0.1524" layer="20" curve="-90"/>
 <wire x1="2.54" y1="43.434" x2="2.54" y2="58.166" width="0.1524" layer="20"/>
-<wire x1="44.196" y1="8.636" x2="44.196" y2="25.908" width="0.1524" layer="20"/>
+<wire x1="44.196" y1="7.366" x2="44.196" y2="25.908" width="0.1524" layer="20"/>
 <wire x1="44.196" y1="25.908" x2="45.72" y2="27.432" width="0.1524" layer="20" curve="-90"/>
 <wire x1="45.72" y1="27.432" x2="50.8" y2="27.432" width="0.1524" layer="20"/>
@@
 <wire x1="50.546" y1="6.096" x2="45.466" y2="6.096" width="0.1524" layer="20"/>
 <wire x1="45.466" y1="6.096" x2="44.196" y2="7.366" width="0.1524" layer="20" curve="-90"/>
-<wire x1="44.196" y1="7.366" x2="44.196" y2="8.636" width="0.1524" layer="20"/>
 </plain>
 <attributes>
@@
 <attribute name="PRICE" value="None" x="6.604" y="48.768" size="1.778" layer="27" display="off"/>
 </element>
-<element name="U$1" library="Adafruit-PowerBoost-FYDE" package="ADAFRUITPOWERBOOSTER(FYDE)" value="ADAFRUITPOWERBOOSTER(FYDE)" x="36.83" y="5.588" rot="R90"/>
 <element name="U1" library="MCU-MCP3008-I_P_DIP16-7.62MM_" package="DIP16-2.54-19.2X7.62MM" value="MCU-MCP3008-I/P(DIP16-7.62MM)" x="27.94" y="45.466">
 <attribute name="AVAILABILITY" value="Unavailable" x="27.94" y="45.466" size="1.778" layer="27" display="off"/>
@@
 </element>
 <element name="X1" library="raspberrypi_bastelstube_v13" package="RASPI_BOARD_B+HAT_DF_CF" value="RASPI_BOARD_B+_HDC" x="2.54" y="5.08"/>
+<element name="U$2" library="MT3608" package="MT3608" value="MT3608" x="13.462" y="6.35"/>
+<element name="J1" library="SparkFun-Connectors" library_urn="urn:adsk.eagle:library:513" package="JST-2-SMD" package3d_urn="urn:adsk.eagle:package:38042/1" value="" x="9.652" y="17.78" rot="R270">
+<attribute name="PROD_ID" value="CONN-11443" x="9.652" y="17.78" size="1.778" layer="27" rot="R270" display="off"/>
+<attribute name="SF_ID" value="PRT-08612" x="9.652" y="17.78" size="1.778" layer="27" rot="R270" display="off"/>
+</element>
 </elements>
 <signals>
@@
 <contactref element="X1" pad="6"/>
 <polygon width="0.3048" layer="16">
-<vertex x="-2.794" y="67.31"/>
-<vertex x="-2.794" y="36.322"/>
-<vertex x="51.308" y="36.322"/>
-<vertex x="51.308" y="67.31"/>
+<vertex x="3.048" y="60.706"/>
+<vertex x="3.556" y="5.08"/>
+<vertex x="43.18" y="5.08"/>
+<vertex x="42.672" y="60.706"/>
 </polygon>
+<contactref element="U$2" pad="P$2"/>
+<contactref element="U$2" pad="P$4"/>
+<contactref element="J1" pad="1"/>
+<wire x1="5.952" y1="18.78" x2="12.462" y2="18.78" width="1.27" layer="1"/>
+<wire x1="12.462" y1="18.78" x2="15.494" y2="15.748" width="1.27" layer="1"/>
+<wire x1="15.494" y1="15.748" x2="15.494" y2="7.874" width="1.27" layer="1"/>
 </signal>
 <signal name="+3V3A">
@@
 <contactref element="U1" pad="15"/>
 <contactref element="X1" pad="1"/>
-<wire x1="10.91" y1="56.31" x2="17.944" y2="49.276" width="1.016" layer="1"/>
+<wire x1="10.91" y1="56.31" x2="15.576" y2="51.644" width="1.016" layer="1"/>
+<wire x1="15.576" y1="51.644" x2="17.944" y2="49.276" width="1.016" layer="1"/>
 <wire x1="17.944" y1="49.276" x2="19.05" y2="49.276" width="1.016" layer="1"/>
 <wire x1="19.05" y1="49.276" x2="21.59" y2="49.276" width="1.016" layer="1"/>
+<contactref element="U$2" pad="P$1"/>
+<contactref element="J1" pad="2"/>
+<wire x1="15.576" y1="51.644" x2="15.576" y2="43.77" width="1.016" layer="1"/>
+<wire x1="15.576" y1="43.77" x2="15.494" y2="43.688" width="1.016" layer="1"/>
+<via x="15.494" y="43.688" extent="1-16" drill="1"/>
+<wire x1="15.494" y1="43.688" x2="15.494" y2="21.844" width="1.016" layer="16"/>
+<wire x1="5.952" y1="16.78" x2="10.144" y2="16.78" width="1.016" layer="1"/>
+<wire x1="10.144" y1="16.78" x2="10.16" y2="16.764" width="1.016" layer="1"/>
+<via x="10.16" y="16.764" extent="1-16" drill="1.016"/>
+<wire x1="10.16" y1="16.764" x2="10.414" y2="16.764" width="1.016" layer="16"/>
+<wire x1="10.414" y1="16.764" x2="15.494" y2="21.844" width="1.016" layer="16"/>
 </signal>
 <signal name="CLK">
@@
 <wire x1="8.7358" y1="56.4633625" x2="8.7358" y2="56.6758" width="0.6096" layer="1"/>
 <wire x1="8.7358" y1="56.6758" x2="10.91" y2="58.85" width="0.6096" layer="1"/>
-<wire x1="8.636" y1="50.8" x2="8.636" y2="56.3635625" width="0.6096" layer="1"/>
+<wire x1="8.636" y1="50.8" x2="8.636" y2="51.816" width="0.6096" layer="1"/>
+<contactref element="U$2" pad="P$3"/>
+<wire x1="8.636" y1="51.816" x2="8.636" y2="56.3635625" width="0.6096" layer="1"/>
+<wire x1="8.636" y1="51.816" x2="12.954" y2="47.498" width="0.6096" layer="1"/>
+<wire x1="12.954" y1="47.498" x2="12.954" y2="43.688" width="0.6096" layer="1"/>
+<via x="12.954" y="43.688" extent="1-16" drill="0.6096"/>
+<wire x1="12.954" y1="43.688" x2="12.954" y2="33.274" width="0.6096" layer="16"/>
+<via x="12.954" y="33.274" extent="1-16" drill="0.6096"/>
+<wire x1="12.954" y1="33.274" x2="20.574" y2="25.654" width="0.6096" layer="1"/>
+<wire x1="20.574" y1="25.654" x2="34.798" y2="25.654" width="0.6096" layer="1"/>
+<wire x1="34.798" y1="25.654" x2="37.846" y2="25.654" width="0.6096" layer="1"/>
+<wire x1="37.846" y1="25.654" x2="41.656" y2="21.844" width="0.6096" layer="1"/>
 </signal>
 <signal name="CS">
@@
 </board>
 </drawing>
+<compatibility>
+<note version="8.2" severity="warning">
+Since Version 8.2, EAGLE supports online libraries. The ids
+of those online libraries will not be understood (or retained)
+with this version.
+</note>
+<note version="8.3" severity="warning">
+Since Version 8.3, EAGLE supports URNs for individual library
+assets (packages, symbols, and devices). The URNs of those assets
+will not be understood (or retained) with this version.
+</note>
+<note version="8.3" severity="warning">
+Since Version 8.3, EAGLE supports the association of 3D packages
+with devices in libraries, schematics, and board files. Those 3D
+packages will not be understood (or retained) with this version.
+</note>
+</compatibility>
 </eagle>

Commit message: Add files via upload
Parts:
- removed J1: (no value), SparkFun-Connectors:JST-2-SMD
- added J2: (no value), SparkFun-Connectors:JST-2-SMD
Connections:
- new net VBAT: J2.2, U$2.P$1
- net +3V3A: no longer J1.2, U$2.P$1
- net GND: now also J2.1; no longer J1.1
Routing:
- net +3V3A: track 55.1 -> 13.6 mm, vias 2 -> 0
- net GND: track 18.7 -> 11.5 mm
- net VBAT: track 0.00 -> 5.99 mm
Changed lines of the file:
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@@
 <layer number="115" name="ReferenceISLANDS" color="7" fill="1" visible="yes" active="yes"/>
 <layer number="116" name="Patch_BOT" color="9" fill="4" visible="no" active="yes"/>
+<layer number="117" name="BACKMAAT1" color="7" fill="1" visible="yes" active="yes"/>
 <layer number="118" name="Rect_Pads" color="7" fill="1" visible="no" active="no"/>
+<layer number="119" name="KAP_TEKEN" color="7" fill="1" visible="yes" active="yes"/>
+<layer number="120" name="KAP_MAAT1" color="7" fill="1" visible="yes" active="yes"/>
 <layer number="121" name="sName" color="7" fill="1" visible="no" active="yes"/>
 <layer number="122" name="_bPlace" color="7" fill="1" visible="no" active="yes"/>
@@
 <layer number="128" name="_bValues" color="7" fill="1" visible="no" active="yes"/>
 <layer number="129" name="Mask" color="7" fill="1" visible="yes" active="yes"/>
+<layer number="130" name="SMDSTROOK" color="7" fill="1" visible="yes" active="yes"/>
 <layer number="131" name="tAdjust" color="7" fill="1" visible="no" active="yes"/>
 <layer number="132" name="bAdjust" color="7" fill="1" visible="no" active="yes"/>
+<layer number="133" name="bottom_silk" color="7" fill="1" visible="yes" active="yes"/>
+<layer number="134" name="silk_top" color="7" fill="1" visible="yes" active="yes"/>
+<layer number="135" name="silk_bottom" color="7" fill="1" visible="yes" active="yes"/>
+<layer number="136" name="silktop" color="7" fill="1" visible="yes" active="yes"/>
+<layer number="137" name="silkbottom" color="7" fill="1" visible="yes" active="yes"/>
 <layer number="144" name="Drill_legend" color="7" fill="1" visible="no" active="yes"/>
+<layer number="145" name="DrillLegend_01-16" color="7" fill="1" visible="yes" active="yes"/>
+<layer number="146" name="DrillLegend_01-20" color="7" fill="1" visible="yes" active="yes"/>
 <layer number="150" name="Notes" color="7" fill="1" visible="no" active="yes"/>
 <layer number="151" name="HeatSink" color="7" fill="1" visible="no" active="yes"/>
@@
 <element name="X1" library="raspberrypi_bastelstube_v13" package="RASPI_BOARD_B+HAT_DF_CF" value="RASPI_BOARD_B+_HDC" x="2.54" y="5.08"/>
 <element name="U$2" library="MT3608" package="MT3608" value="MT3608" x="13.462" y="6.35"/>
-<element name="J1" library="SparkFun-Connectors" library_urn="urn:adsk.eagle:library:513" package="JST-2-SMD" package3d_urn="urn:adsk.eagle:package:38042/1" value="" x="9.652" y="17.78" rot="R270">
-<attribute name="PROD_ID" value="CONN-11443" x="9.652" y="17.78" size="1.778" layer="27" rot="R270" display="off"/>
-<attribute name="SF_ID" value="PRT-08612" x="9.652" y="17.78" size="1.778" layer="27" rot="R270" display="off"/>
+<element name="J2" library="SparkFun-Connectors" library_urn="urn:adsk.eagle:library:513" package="JST-2-SMD" package3d_urn="urn:adsk.eagle:package:38042/1" value="" x="6.858" y="18.288" rot="R90">
+<attribute name="PROD_ID" value="CONN-11443" x="-9.144" y="9.398" size="1.778" layer="27" rot="R90" display="off"/>
+<attribute name="SF_ID" value="PRT-08612" x="-9.144" y="9.398" size="1.778" layer="27" rot="R90" display="off"/>
 </element>
 </elements>
@@
 <contactref element="U$2" pad="P$2"/>
 <contactref element="U$2" pad="P$4"/>
-<contactref element="J1" pad="1"/>
-<wire x1="5.952" y1="18.78" x2="12.462" y2="18.78" width="1.27" layer="1"/>
-<wire x1="12.462" y1="18.78" x2="15.494" y2="15.748" width="1.27" layer="1"/>
-<wire x1="15.494" y1="15.748" x2="15.494" y2="7.874" width="1.27" layer="1"/>
+<contactref element="J2" pad="1"/>
+<wire x1="10.558" y1="17.288" x2="15.494" y2="12.352" width="1.524" layer="1"/>
+<wire x1="15.494" y1="12.352" x2="15.494" y2="7.874" width="1.524" layer="1"/>
 </signal>
 <signal name="+3V3A">
@@
 <wire x1="17.944" y1="49.276" x2="19.05" y2="49.276" width="1.016" layer="1"/>
 <wire x1="19.05" y1="49.276" x2="21.59" y2="49.276" width="1.016" layer="1"/>
-<contactref element="U$2" pad="P$1"/>
-<contactref element="J1" pad="2"/>
-<wire x1="15.576" y1="51.644" x2="15.576" y2="43.77" width="1.016" layer="1"/>
-<wire x1="15.576" y1="43.77" x2="15.494" y2="43.688" width="1.016" layer="1"/>
-<via x="15.494" y="43.688" extent="1-16" drill="1"/>
-<wire x1="15.494" y1="43.688" x2="15.494" y2="21.844" width="1.016" layer="16"/>
-<wire x1="5.952" y1="16.78" x2="10.144" y2="16.78" width="1.016" layer="1"/>
-<wire x1="10.144" y1="16.78" x2="10.16" y2="16.764" width="1.016" layer="1"/>
-<via x="10.16" y="16.764" extent="1-16" drill="1.016"/>
-<wire x1="10.16" y1="16.764" x2="10.414" y2="16.764" width="1.016" layer="16"/>
-<wire x1="10.414" y1="16.764" x2="15.494" y2="21.844" width="1.016" layer="16"/>
 </signal>
 <signal name="CLK">
@@
 <wire x1="34.29" y1="51.054" x2="34.29" y2="49.276" width="1.016" layer="1"/>
 </signal>
+<signal name="VBAT">
+<contactref element="U$2" pad="P$1"/>
+<contactref element="J2" pad="2"/>
+<wire x1="15.494" y1="21.844" x2="12.938" y2="19.288" width="1.143" layer="1"/>
+<wire x1="12.938" y1="19.288" x2="10.558" y2="19.288" width="1.143" layer="1"/>
+</signal>
 </signals>
